Commit message: inertia modified

File: models/panda/panda.urdf (robot description, URDF)
Before this commit: robot panda, 8 links, 7 joints
Links:
- link panda_link0: mass 3.06 -> 2.8142028896
- link panda_link1: mass 2.34 -> 2.3599995791
- link panda_link2: mass 2.36 -> 2.379518833
- link panda_link3: mass 2.38 -> 2.6498823337
- link panda_link4: mass 2.43 -> 2.6948018744
- link panda_link5: mass 3.5 -> 2.9812816864
- link panda_link6: mass 1.47 -> 1.1285806309
- link panda_link7: mass 0.45 -> 0.4052912465

File: models/panda/panda_gripper.urdf (robot description, URDF)
Before this commit: robot panda, 12 links, 11 joints
Links:
- removed link panda_link8
Joints:
- removed joint panda_joint8
- joint panda_hand_joint: origin xyz=0 0 0 rpy=0 0 -0.785398163397 -> xyz=0 0 0.107 rpy=0 0 -0.785398163397; parent panda_link8 -> panda_link7
- joint panda_joint1: limit lower=-2.9671 upper=2.9671 effort=87 velocity=2.1750 -> lower=-2.8973 upper=2.8973 effort=87 velocity=2.1750
- joint panda_joint2: limit lower=-1.8326 upper=1.8326 effort=87 velocity=2.1750 -> lower=-1.7628 upper=1.7628 effort=87 velocity=2.1750
- joint panda_joint3: limit lower=-2.9671 upper=2.9671 effort=87 velocity=2.1750 -> lower=-2.8973 upper=2.8973 effort=87 velocity=2.1750
- joint panda_joint4: limit lower=-3.1416 upper=0.0 effort=87 velocity=2.1750 -> lower=-3.0718 upper=-0.0698 effort=87 velocity=2.1750
- joint panda_joint5: limit lower=-2.9671 upper=2.9671 effort=12 velocity=2.6100 -> lower=-2.8973 upper=2.8973 effort=12 velocity=2.6100
- joint panda_joint6: limit lower=-0.0873 upper=3.8223 effort=12 velocity=2.6100 -> lower=-0.0175 upper=3.752 effort=12 velocity=2.6100
- joint panda_joint7: limit lower=-2.9671 upper=2.9671 effort=12 velocity=2.6100 -> lower=-2.8973 upper=2.8973 effort=12 velocity=2.6100

Commit message: inverse dynamics and kinematics added with examples

File: models/panda/panda.urdf (robot description, URDF)
Before this commit: robot panda, 8 links, 7 joints
Links:
- added link panda_EndEffector
Joints:
- added joint panda_joint8: type fixed, parent panda_link7, child panda_EndEffector, origin xyz=0 0 0.107 rpy=0 0 0, axis 0 0 0
